Commit message: fixed bug gazebo launch file
changing name of package in ROS to explo bot2

File: src/explo_bot2/urdf/explo_bot.xacro (robot description, xacro)
@@ -34,5 +34,5 @@
       <origin xyz="0 0 0.35" rpy=" 0 0 0"/>
       <geometry>
-        <box size="0.2 0.2 0.8"/>
+        <box size="0.2 0.2 0.55"/>
       </geometry>
     </collision>
@@ -40,9 +40,9 @@
       <origin xyz="0 0 0.35" rpy=" 0 0 0"/>
       <geometry>
-        <box size="0.2 0.2 0.8"/>
+        <box size="0.2 0.2 0.55"/>
       </geometry>
     </visual>
     <collision name='left_arm'>
-      <origin xyz="0.1 0.15 0.35" rpy=" 0 0 0"/>
+      <origin xyz="0.1 0.15 0.25" rpy=" 0 0 0"/>
       <geometry>
         <box size="0.2 0.1 0.1"/>
@@ -50,5 +50,5 @@
     </collision>
     <visual name='left_arm_visual'>
-      <origin xyz="0.1 0.15 0.35" rpy=" 0 0 0"/>
+      <origin xyz="0.1 0.15 0.25" rpy=" 0 0 0"/>
       <geometry>
         <box size="0.2 0.1 0.1"/>
@@ -56,5 +56,5 @@
     </visual>
     <collision name='right_arm'>
-      <origin xyz="0.1 -0.15 0.35" rpy=" 0 0 0"/>
+      <origin xyz="0.1 -0.15 0.25" rpy=" 0 0 0"/>
       <geometry>
         <box size="0.2 0.1 0.1"/>
@@ -62,5 +62,5 @@
     </collision>
     <visual name='right_arm_visual'>
-      <origin xyz="0.1 -0.15 0.35" rpy=" 0 0 0"/>
+      <origin xyz="0.1 -0.15 0.25" rpy=" 0 0 0"/>
       <geometry>
         <box size="0.2 0.1 0.1"/>

Commit message: fixed bug with package name

File: src/explo_bot2/urdf/explo_bot.xacro (robot description, xacro)
@@ -34,5 +34,5 @@
       <origin xyz="0 0 0.35" rpy=" 0 0 0"/>
       <geometry>
-        <box size="0.2 0.2 0.55"/>
+        <box size="0.2 0.2 0.40"/>
       </geometry>
     </collision>
@@ -40,9 +40,9 @@
       <origin xyz="0 0 0.35" rpy=" 0 0 0"/>
       <geometry>
-        <box size="0.2 0.2 0.55"/>
+        <box size="0.2 0.2 0.40"/>
       </geometry>
     </visual>
     <collision name='left_arm'>
-      <origin xyz="0.1 0.15 0.25" rpy=" 0 0 0"/>
+      <origin xyz="0.1 0.15 0.2" rpy=" 0 0 0"/>
       <geometry>
         <box size="0.2 0.1 0.1"/>
@@ -50,5 +50,5 @@
     </collision>
     <visual name='left_arm_visual'>
-      <origin xyz="0.1 0.15 0.25" rpy=" 0 0 0"/>
+      <origin xyz="0.1 0.15 0.2" rpy=" 0 0 0"/>
       <geometry>
         <box size="0.2 0.1 0.1"/>
@@ -56,5 +56,5 @@
     </visual>
     <collision name='right_arm'>
-      <origin xyz="0.1 -0.15 0.25" rpy=" 0 0 0"/>
+      <origin xyz="0.1 -0.15 0.2" rpy=" 0 0 0"/>
       <geometry>
         <box size="0.2 0.1 0.1"/>
@@ -62,5 +62,5 @@
     </collision>
     <visual name='right_arm_visual'>
-      <origin xyz="0.1 -0.15 0.25" rpy=" 0 0 0"/>
+      <origin xyz="0.1 -0.15 0.2" rpy=" 0 0 0"/>
       <geometry>
         <box size="0.2 0.1 0.1"/>

Commit message: removing hokuyo sensor

File: src/explo_bot2/urdf/explo_bot.xacro (robot description, xacro)
@@ -185,32 +185,3 @@
 	    <parent link="chassis"/>
   </joint>
-  <link name='hokuyo'>
-	  <pose>0 0 0.1 0 0 0</pose>
-	  <inertial>
-	      <mass value="0.1"/>
-	      <origin xyz="0 0 0" rpy="0 0 0"/>
-	      <inertia
-		  ixx="1e-6" ixy="0" ixz="0"
-		  iyy="1e-6" iyz="0"
-		  izz="1e-6"
-	      />
-	    </inertial>
-	    <collision name='hokuyo_collision'>
-	      <origin xyz="0 0 0" rpy=" 0 0 0"/>
-	      <geometry>
-		<box size="0.01 0.01 0.01"/>
-	      </geometry>
-	    </collision>
-	    <visual name='hokuyo_visual'>
-	      <origin xyz="0 0 0" rpy=" 0 0 0"/>
-	      <geometry>
-		<mesh filename="$(find explo_bot)/meshes/hokuyo.dae"/>
-	      </geometry>
-	    </visual>
-  </link>
-  <joint type="fixed" name="hokuyo_joint">
-	    <origin xyz="0.15 0 0.15" rpy="0 0 0"/>
-	    <child link="hokuyo"/>
-	    <parent link="chassis"/>
-  </joint>
 </robot>

Commit message: modified z position of arms

File: src/explo_bot2/urdf/explo_bot.xacro (robot description, xacro)
@@ -44,5 +44,5 @@
     </visual>
     <collision name='left_arm'>
-      <origin xyz="0.1 0.15 0.2" rpy=" 0 0 0"/>
+      <origin xyz="0.1 0.15 0.25" rpy=" 0 0 0"/>
       <geometry>
         <box size="0.2 0.1 0.1"/>
@@ -50,5 +50,5 @@
     </collision>
     <visual name='left_arm_visual'>
-      <origin xyz="0.1 0.15 0.2" rpy=" 0 0 0"/>
+      <origin xyz="0.1 0.15 0.25" rpy=" 0 0 0"/>
       <geometry>
         <box size="0.2 0.1 0.1"/>
@@ -56,5 +56,5 @@
     </visual>
     <collision name='right_arm'>
-      <origin xyz="0.1 -0.15 0.2" rpy=" 0 0 0"/>
+      <origin xyz="0.1 -0.15 0.25" rpy=" 0 0 0"/>
       <geometry>
         <box size="0.2 0.1 0.1"/>
@@ -62,5 +62,5 @@
     </collision>
     <visual name='right_arm_visual'>
-      <origin xyz="0.1 -0.15 0.2" rpy=" 0 0 0"/>
+      <origin xyz="0.1 -0.15 0.25" rpy=" 0 0 0"/>
       <geometry>
         <box size="0.2 0.1 0.1"/>

Commit message: adding hokuyo sensor

File: src/explo_bot2/urdf/explo_bot.xacro (robot description, xacro)
@@ -185,3 +185,32 @@
 	    <parent link="chassis"/>
   </joint>
+  <link name='hokuyo'>
+	  <pose>0 0 0.1 0 0 0</pose>
+	  <inertial>
+	      <mass value="0.1"/>
+	      <origin xyz="0 0 0" rpy="0 0 0"/>
+	      <inertia
+		  ixx="1e-6" ixy="0" ixz="0"
+		  iyy="1e-6" iyz="0"
+		  izz="1e-6"
+	      />
+	    </inertial>
+	    <collision name='hokuyo_collision'>
+	      <origin xyz="0 0 0" rpy=" 0 0 0"/>
+	      <geometry>
+		<box size="0.01 0.01 0.01"/>
+	      </geometry>
+	    </collision>
+	    <visual name='hokuyo_visual'>
+	      <origin xyz="0 0 0" rpy=" 0 0 0"/>
+	      <geometry>
+		<mesh filename="$(find explo_bot)/meshes/hokuyo.dae"/>
+	      </geometry>
+	    </visual>
+  </link>
+  <joint type="fixed" name="hokuyo_joint">
+	    <origin xyz="0.15 0 0.15" rpy="0 0 0"/>
+	    <child link="hokuyo"/>
+	    <parent link="chassis"/>
+  </joint>
 </robot>

Commit message: changed camera from RGB to RGBD

File: src/explo_bot2/urdf/explo_bot.xacro (robot description, xacro)
@@ -32,37 +32,37 @@
     </visual>
     <collision name='center_box'>
-      <origin xyz="0 0 0.35" rpy=" 0 0 0"/>
-      <geometry>
-        <box size="0.2 0.2 0.40"/>
+      <origin xyz="0 0 0.175" rpy=" 0 0 0"/>
+      <geometry>
+        <box size="0.15 0.15 0.2"/>
       </geometry>
     </collision>
     <visual name='center_box_visual'>
-      <origin xyz="0 0 0.35" rpy=" 0 0 0"/>
-      <geometry>
-        <box size="0.2 0.2 0.40"/>
+      <origin xyz="0 0 0.175" rpy=" 0 0 0"/>
+      <geometry>
+        <box size="0.15 0.15 0.2"/>
       </geometry>
     </visual>
     <collision name='left_arm'>
-      <origin xyz="0.1 0.15 0.25" rpy=" 0 0 0"/>
-      <geometry>
-        <box size="0.2 0.1 0.1"/>
+      <origin xyz="0.05 0.1 0.17" rpy=" 0 0 0"/>
+      <geometry>
+        <box size="0.14 0.05 0.05"/>
       </geometry>
     </collision>
     <visual name='left_arm_visual'>
-      <origin xyz="0.1 0.15 0.25" rpy=" 0 0 0"/>
-      <geometry>
-        <box size="0.2 0.1 0.1"/>
+      <origin xyz="0.05 0.1 0.17" rpy=" 0 0 0"/>
+      <geometry>
+        <box size="0.14 0.05 0.05"/>
       </geometry>
     </visual>
     <collision name='right_arm'>
-      <origin xyz="0.1 -0.15 0.25" rpy=" 0 0 0"/>
-      <geometry>
-        <box size="0.2 0.1 0.1"/>
+      <origin xyz="0.05 -0.1 0.17" rpy=" 0 0 0"/>
+      <geometry>
+        <box size="0.14 0.05 0.05"/>
       </geometry>
     </collision>
     <visual name='right_arm_visual'>
-      <origin xyz="0.1 -0.15 0.25" rpy=" 0 0 0"/>
-      <geometry>
-        <box size="0.2 0.1 0.1"/>
+      <origin xyz="0.05 -0.1 0.17" rpy=" 0 0 0"/>
+      <geometry>
+        <box size="0.14 0.05 0.05"/>
       </geometry>
     </visual>
@@ -181,5 +181,5 @@
   </link>
   <joint type="fixed" name="camera_joint">
-	    <origin xyz="0.1 0 0.5" rpy="0 0 0"/>
+	    <origin xyz="0.18 0 0.1" rpy="0 0 0"/>
 	    <child link="camera"/>
 	    <parent link="chassis"/>
@@ -210,5 +210,5 @@
   </link>
   <joint type="fixed" name="hokuyo_joint">
-	    <origin xyz="0.15 0 0.15" rpy="0 0 0"/>
+	    <origin xyz="0.05 0 0.32" rpy="0 0 0"/>
 	    <child link="hokuyo"/>
 	    <parent link="chassis"/>
