Commit message: catkin

File: src/slam_project/urdf/explo_bot.xacro (robot description, xacro)
@@ -1,5 +1,5 @@
 <?xml version='1.0'?>
 <robot name="explo_bot" xmlns:xacro="http://www.ros.org/wiki/xacro">
-  <xacro:include filename="$(find explo_bot2)/urdf/explo_bot.gazebo" />
+  <xacro:include filename="$(find slam_project)/urdf/explo_bot.gazebo" />
   <link name="robot_footprint"></link>
   <joint name="robot_footprint_joint" type="fixed">
@@ -180,8 +180,14 @@
 	    </visual>
   </link>
-  <joint type="fixed" name="camera_joint">
+  <joint type="fixed" name="camera_joint2">
 	    <origin xyz="0.18 0 0.1" rpy="0 0 0"/>
 	    <child link="camera"/>
 	    <parent link="chassis"/>
+  </joint>
+  <link name="camera_rgbd_frame"/>
+  <joint name="camera_joint" type="fixed">
+      <origin xyz="0 0 0" rpy="-1.5707 0 -1.5707"/>
+      <parent link="camera"/>
+      <child link="camera_rgbd_frame"/>
   </joint>
   <link name='hokuyo'>

Commit message: position of camera joint fixed

File: src/slam_project/urdf/explo_bot.xacro (robot description, xacro)
@@ -185,9 +185,14 @@
 	    <parent link="chassis"/>
   </joint>
-  <link name="camera_rgbd_frame"/>
   <joint name="camera_joint" type="fixed">
-      <origin xyz="0 0 0" rpy="-1.5707 0 -1.5707"/>
+      <origin xyz="0.18 0 0.1" rpy="-1.5707 0 -1.5707"/>
       <parent link="camera"/>
       <child link="camera_rgbd_frame"/>
+  </joint>
+ <link name="camera_rgbd_frame"/>
+  <joint type="fixed" name="camera_joint3">
+	<origin xyz="0.18 0 0.1" rpy="0 0 0"/>
+	<child link="camera_rgbd_frame"/>
+	<parent link="chassis"/>
   </joint>
   <link name='hokuyo'>

Commit message: BUG camera topics

File: src/slam_project/urdf/explo_bot.xacro (robot description, xacro)
@@ -190,10 +190,5 @@
       <child link="camera_rgbd_frame"/>
   </joint>
- <link name="camera_rgbd_frame"/>
-  <joint type="fixed" name="camera_joint3">
-	<origin xyz="0.18 0 0.1" rpy="0 0 0"/>
-	<child link="camera_rgbd_frame"/>
-	<parent link="chassis"/>
-  </joint>
+ <link name="camera_rgbd_frame"> </link>
   <link name='hokuyo'>
 	  <pose>0 0 0.1 0 0 0</pose>

Commit message: change name for base footprint

File: src/slam_project/urdf/explo_bot.xacro (robot description, xacro)
@@ -2,8 +2,8 @@
 <robot name="explo_bot" xmlns:xacro="http://www.ros.org/wiki/xacro">
   <xacro:include filename="$(find slam_project)/urdf/explo_bot.gazebo" />
-  <link name="robot_footprint"></link>
+  <link name="base_footprint"></link>
   <joint name="robot_footprint_joint" type="fixed">
     <origin xyz="0 0 0" rpy="0 0 0" />
-    <parent link="robot_footprint"/>
+    <parent link="base_footprint"/>
     <child link="chassis" />
   </joint>
@@ -176,5 +176,5 @@
 	      <origin xyz="0 0 0" rpy=" 0 0 0"/>
 	      <geometry>
-		<box size="0.05 0.05 0.05"/>
+		<mesh filename="$(find slam_project)/meshes/kinect.dae"/>
 	      </geometry>
 	    </visual>
@@ -211,5 +211,5 @@
 	      <origin xyz="0 0 0" rpy=" 0 0 0"/>
 	      <geometry>
-		<mesh filename="$(find explo_bot)/meshes/hokuyo.dae"/>
+		<mesh filename="$(find slam_project)/meshes/hokuyo.dae"/>
 	      </geometry>
 	    </visual>

Commit message: base footprint update

File: src/slam_project/urdf/explo_bot.xacro (robot description, xacro)
@@ -2,8 +2,8 @@
 <robot name="explo_bot" xmlns:xacro="http://www.ros.org/wiki/xacro">
   <xacro:include filename="$(find slam_project)/urdf/explo_bot.gazebo" />
-  <link name="base_footprint"></link>
+  <link name="robot_footprint"></link>
   <joint name="robot_footprint_joint" type="fixed">
     <origin xyz="0 0 0" rpy="0 0 0" />
-    <parent link="base_footprint"/>
+    <parent link="robot_footprint"/>
     <child link="chassis" />
   </joint>
